File: pcb/lazercut.kicad_pcb (KiCad board)
At the start: 2 copper layers, 354.2 x 117.1 mm, 145 parts, among them SW1 SW_Push, SW10 SW_Push, SW11 SW_Push, SW12 SW_Push, SW13 SW_Push, SW14 SW_Push, SW15 SW_Push, SW16 SW_Push, SW17 SW_Push, SW18 SW_Push, SW19 SW_Push, SW2 SW_Push, SW20 SW_Push, SW21 SW_Push, SW22 SW_Push, SW23 SW_Push, SW24 SW_Push, SW25 SW_Push, SW26 SW_Push, SW27 SW_Push, SW28 SW_Push, SW29 SW_Push, SW3 SW_Push, SW30 SW_Push, SW31 SW_Push, SW32 SW_Push, SW33 SW_Push, SW34 SW_Push, SW35 SW_Push, SW36 SW_Push, SW37 SW_Push, SW38 SW_Push, SW39 SW_Push, SW4 SW_Push, SW40 SW_Push, SW41 SW_Push, SW42 SW_Push, SW43 SW_Push, SW44 SW_Push, SW45 SW_Push, SW46 SW_Push, SW47 SW_Push, SW48 SW_Push, SW49 SW_Push, SW5 SW_Push, SW50 SW_Push, SW51 SW_Push, SW52 SW_Push, SW53 SW_Push, SW54 SW_Push, SW55 SW_Push, SW56 SW_Push, SW57 SW_Push, SW58 SW_Push, SW59 SW_Push, SW6 SW_Push, SW60 SW_Push, SW61 SW_Push, SW62 SW_Push, SW63 SW_Push, SW64 SW_Push, SW65 SW_Push, SW66 SW_Push, SW67 SW_Push, SW68 SW_Push, SW69 SW_Push, SW7 SW_Push, SW70 SW_Push, SW71 SW_Push, SW72 SW_Push, SW8 SW_Push, SW9 SW_Push, U1 Elite-C

Commit message: re do pcb aligment and traceing
Parts:
- U1: footprint Keebio-Parts:Elite-C-castellated-29pin-holes -> Keebio-Parts:Elite-C
- moved D72 4.76 mm to (349.2, 114.8)
- moved SW71 4.76 mm to (325.0, 110.7)
- moved D70 4.76 mm to (311.1, 114.8)
- moved D71 4.76 mm to (330.1, 114.8)
- moved SW70 4.76 mm to (306.0, 110.7)
- moved SW72 4.76 mm to (344.1, 110.7)
Routing:
- net col0: track 389.7 -> 302.2 mm, vias 1 -> 0
- net row4: track 586.5 -> 508.6 mm, vias 2 -> 0
- net col1: track 272.0 -> 196.2 mm
- net col4: track 308.2 -> 380.4 mm, vias 3 -> 1
- net col2: track 365.0 -> 305.8 mm, vias 4 -> 1
- net row3: track 455.8 -> 506.9 mm, vias 2 -> 0
- net row5: track 570.7 -> 533.8 mm
- net col7: track 318.5 -> 349.4 mm, vias 2 -> 1
- net row0: track 534.4 -> 505.6 mm
- net col5: track 366.8 -> 339.4 mm, vias 2 -> 1
- net row2: track 461.1 -> 445.9 mm
- net col3: track 241.7 -> 228.8 mm
- net row6: track 505.8 -> 492.9 mm
- net row7: track 512.0 -> 502.5 mm
- net col8: track 233.6 -> 240.5 mm
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Other:
- board size 354.2 x 117.1 mm -> 338.6 x 105.3 mm

Commit message: reposition elite-c because of outer frame
Parts:
- moved U1 0.55 mm to (335.3, 72.6)
Routing:
- net col4: track 380.4 -> 288.0 mm
- net row3: track 506.9 -> 450.5 mm
- net col3: track 228.8 -> 185.3 mm
- net row0: track 505.6 -> 540.3 mm
- net col8: track 240.5 -> 270.4 mm
- net col7: track 349.4 -> 325.0 mm, vias 1 -> 0
- net col5: track 339.4 -> 363.8 mm, vias 1 -> 0
- net row2: track 445.9 -> 465.8 mm, vias 1 -> 3
- net row1: track 514.2 -> 532.8 mm, vias 1 -> 0
- net row5: track 533.8 -> 550.5 mm, vias 1 -> 0
- net col1: track 196.2 -> 184.1 mm
- net row4: track 508.6 -> 502.8 mm, vias 0 -> 1
- net row7: track 502.5 -> 508.2 mm, vias 0 -> 1
- net row6: track 492.9 -> 489.0 mm
- net col2: track 305.8 -> 303.8 mm
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