File: pcb/lasercut.kicad_sch (KiCad schematic)
At the start: 145 parts, among them SW1 SW_Push, SW10 SW_Push, SW11 SW_Push, SW12 SW_Push, SW13 SW_Push, SW14 SW_Push, SW15 SW_Push, SW16 SW_Push, SW17 SW_Push, SW18 SW_Push, SW19 SW_Push, SW2 SW_Push, SW20 SW_Push, SW21 SW_Push, SW22 SW_Push, SW23 SW_Push, SW24 SW_Push, SW25 SW_Push, SW26 SW_Push, SW27 SW_Push, SW28 SW_Push, SW29 SW_Push, SW3 SW_Push, SW30 SW_Push, SW31 SW_Push, SW32 SW_Push, SW33 SW_Push, SW34 SW_Push, SW35 SW_Push, SW36 SW_Push, SW37 SW_Push, SW38 SW_Push, SW39 SW_Push, SW4 SW_Push, SW40 SW_Push, SW41 SW_Push, SW42 SW_Push, SW43 SW_Push, SW44 SW_Push, SW45 SW_Push, SW46 SW_Push, SW47 SW_Push, SW48 SW_Push, SW49 SW_Push, SW5 SW_Push, SW50 SW_Push, SW51 SW_Push, SW52 SW_Push, SW53 SW_Push, SW54 SW_Push, SW55 SW_Push, SW56 SW_Push, SW57 SW_Push, SW58 SW_Push, SW59 SW_Push, SW6 SW_Push, SW60 SW_Push, SW61 SW_Push, SW62 SW_Push, SW63 SW_Push, SW64 SW_Push, SW65 SW_Push, SW66 SW_Push, SW67 SW_Push, SW68 SW_Push, SW69 SW_Push, SW7 SW_Push, SW70 SW_Push, SW71 SW_Push, SW72 SW_Push, SW8 SW_Push, SW9 SW_Push, U1 Elite-C

Commit message: add batter headers
Parts:
- added J1: Conn_01x02_Male, Connector_PinHeader_2.54mm:PinHeader_1x02_P2.54mm_Horizontal, symbol Connector:Conn_01x02_Male
Connections:
- net GND: now also J1.2 (Pin_2)
- net BAT: now reaches U1.24 (B0)
- net BAT: now also J1.1 (Pin_1)
Changed lines of the file:
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@@
+    (stroke (width 0) (type default) (color 0 0 0 0))
+  )
+  (wire (pts (xy 254 22.86) (xy 259.08 22.86))
     (stroke (width 0) (type default) (color 0 0 0 0))
   )
@@
     )
   )
+  (global_label "BAT" (shape input) (at 254 20.32 0) (fields_autoplaced)
+    (effects (font (size 1.27 1.27)) (justify left))
+    (property "Intersheet References" "${INTERSHEET_REFS}" (id 0) (at 259.6504 20.2406 0)
+      (effects (font (size 1.27 1.27)) (justify left) hide)
+    )
+  )
+  (global_label "BAT" (shape input) (at 265.43 48.26 0) (fields_autoplaced)
+    (effects (font (size 1.27 1.27)) (justify left))
+    (property "Intersheet References" "${INTERSHEET_REFS}" (id 0) (at 271.0804 48.1806 0)
+      (effects (font (size 1.27 1.27)) (justify left) hide)
+    )
+  )
   (global_label "col2" (shape input) (at 265.43 58.42 0) (fields_autoplaced)
     (effects (font (size 1.27 1.27)) (justify left))
@@
     (pin "1")
   )
+  (symbol (lib_id "power:GND") (at 259.08 22.86 0) (unit 1)
+    (in_bom yes) (on_board yes) (fields_autoplaced)
+    (property "Reference" "#PWR01" (id 0) (at 259.08 29.21 0)
+      (effects (font (size 1.27 1.27)) hide)
+    )
+    (property "Value" "GND" (id 1) (at 259.08 27.94 0))
+    (property "Footprint" "" (id 2) (at 259.08 22.86 0)
+      (effects (font (size 1.27 1.27)) hide)
+    )
+    (property "Datasheet" "" (id 3) (at 259.08 22.86 0)
+      (effects (font (size 1.27 1.27)) hide)
+    )
+    (pin "1")
+  )
   (symbol (lib_id "power:GND") (at 276.86 50.8 0) (unit 1)
     (in_bom yes) (on_board yes) (fields_autoplaced)
@@
     )
     (pin "1")
+  )
+  (symbol (lib_id "Connector:Conn_01x02_Male") (at 248.92 20.32 0) (unit 1)
+    (in_bom yes) (on_board yes) (fields_autoplaced)
+    (property "Reference" "J1" (id 0) (at 251.4219 15.24 0))
+    (property "Value" "Conn_01x02_Male" (id 1) (at 251.4219 17.78 0))
+    (property "Footprint" "Connector_PinHeader_2.54mm:PinHeader_1x02_P2.54mm_Horizontal" (id 2) (at 248.92 20.32 0)
+      (effects (font (size 1.27 1.27)) hide)
+    )
+    (property "Datasheet" "~" (id 3) (at 248.92 20.32 0)
+      (effects (font (size 1.27 1.27)) hide)
+    )
+    (pin "1")
+    (pin "2")
   )
   (symbol (lib_id "Device:D") (at 44.45 22.86 0) (unit 1)
@@
   )
   (symbol_instances
+    (path "/5a756ee7-ab2b-41e0-83fe-378fe9f99d39"
+      (reference "#PWR01") (unit 1) (value "GND") (footprint "")
+    )
     (path "/df3c1d99-ef89-4e3d-b257-53ac1ae93e43"
       (reference "#PWR0101") (unit 1) (value "GND") (footprint "")
@@
       (reference "D72") (unit 1) (value "D") (footprint "Diode_SMD:D_SOD-128")
     )
+    (path "/08d2935a-d8e9-4e66-be34-10793b71b57b"
+      (reference "J1") (unit 1) (value "Conn_01x02_Male") (footprint "Connector_PinHeader_2.54mm:PinHeader_1x02_P2.54mm_Horizontal")
+    )
     (path "/00000000-0000-0000-0000-00006179cfaf"

Commit message: new freerouting version
need to redo the matrix/switch position
Parts:
- renumbered D2 to D10, D10 to D11, D18 to D12, D26 to D13, D34 to D14, D42 to D15, D50 to D16, D58 to D17, D66 to D18, D3 to D19, D9 to D2, D11 to D20, D19 to D21, D27 to D22, D35 to D23, D43 to D24, D51 to D25, D59 to D26, D67 to D27, D4 to D28, D12 to D29, D17 to D3, D20 to D30, D28 to D31, D36 to D32, D44 to D33, D52 to D34, D60 to D35, D68 to D36, D5 to D37, D13 to D38, D21 to D39, D25 to D4, D29 to D40, D37 to D41, D45 to D42, D53 to D43, D61 to D44, D69 to D45, D6 to D46, D14 to D47, D22 to D48, D30 to D49, D33 to D5, D38 to D50, D46 to D51, D54 to D52, D62 to D53, D70 to D54, D7 to D55, D15 to D56, D23 to D57, D31 to D58, D39 to D59, D41 to D6, D47 to D60, D55 to D61, D63 to D62, D71 to D63, D8 to D64, D16 to D65, D24 to D66, D32 to D67, D40 to D68, D48 to D69, D49 to D7, D56 to D70, D64 to D71, D57 to D8, D65 to D9, SW2 to SW10, SW10 to SW11, SW18 to SW12, SW26 to SW13, SW34 to SW14, SW42 to SW15, SW50 to SW16, SW58 to SW17, SW66 to SW18, SW3 to SW19, SW9 to SW2, SW11 to SW20, SW19 to SW21, SW27 to SW22, SW35 to SW23, SW43 to SW24, SW51 to SW25, SW59 to SW26, SW67 to SW27, SW4 to SW28, SW12 to SW29, SW17 to SW3, SW20 to SW30, SW28 to SW31, SW36 to SW32, SW44 to SW33, SW52 to SW34, SW60 to SW35, SW68 to SW36, SW5 to SW37, SW13 to SW38, SW21 to SW39, SW25 to SW4, SW29 to SW40, SW37 to SW41, SW45 to SW42, SW53 to SW43, SW61 to SW44, SW69 to SW45, SW6 to SW46, SW14 to SW47, SW22 to SW48, SW30 to SW49, SW33 to SW5, SW38 to SW50, SW46 to SW51, SW54 to SW52, SW62 to SW53, SW70 to SW54, SW7 to SW55, SW15 to SW56, SW23 to SW57, SW31 to SW58, SW39 to SW59, SW41 to SW6, SW47 to SW60, SW55 to SW61, SW63 to SW62, SW71 to SW63, SW8 to SW64, SW16 to SW65, SW24 to SW66, SW32 to SW67, SW40 to SW68, SW48 to SW69, SW49 to SW7, SW56 to SW70, SW64 to SW71, SW57 to SW8, SW65 to SW9
Connections:
- net col2: now also U1.19 (A2/PF5); no longer U1.20 (A3/PF4)
- net col3: now also U1.18 (A1/PF6); no longer U1.19 (A2/PF5)
- net col4: now also U1.17 (A0/PF7); no longer U1.18 (A1/PF6)
- net col5: now also U1.16 (15/PB1); no longer U1.17 (A0/PF7)
- net col6: no longer U1.16 (15/PB1)
- net row0: no longer SW1.1, SW2.1, SW3.1, SW4.1, SW5.1, SW6.1, SW7.1, SW8.1, SW9.1
- net row1: no longer SW10.1, SW11.1, SW12.1, SW13.1, SW14.1, SW15.1, SW16.1, SW17.1, SW18.1
- net row2: no longer SW19.1, SW20.1, SW21.1, SW22.1, SW23.1, SW24.1, SW25.1, SW26.1, SW27.1
- net row3: no longer SW28.1, SW29.1, SW30.1, SW31.1, SW32.1, SW33.1, SW34.1, SW35.1, SW36.1
- net row4: no longer SW37.1, SW38.1, SW39.1, SW40.1, SW41.1, SW42.1, SW43.1, SW44.1, SW45.1
- net row5: no longer SW46.1, SW47.1, SW48.1, SW49.1, SW50.1, SW51.1, SW52.1, SW53.1, SW54.1
- net row6: no longer SW55.1, SW56.1, SW57.1, SW58.1, SW59.1, SW60.1, SW61.1, SW62.1, SW63.1
- net row7: no longer SW64.1, SW65.1, SW66.1, SW67.1, SW68.1, SW69.1, SW70.1, SW71.1, SW72.1
- new net: SW1.1, SW2.1, SW3.1, SW4.1, SW5.1, SW6.1, SW7.1, SW8.1, SW9.1
- new net: SW10.1, SW11.1, SW12.1, SW13.1, SW14.1, SW15.1, SW16.1, SW17.1, SW18.1
- new net: SW19.1, SW20.1, SW21.1, SW22.1, SW23.1, SW24.1, SW25.1, SW26.1, SW27.1
- new net: SW28.1, SW29.1, SW30.1, SW31.1, SW32.1, SW33.1, SW34.1, SW35.1, SW36.1
- new net: SW37.1, SW38.1, SW39.1, SW40.1, SW41.1, SW42.1, SW43.1, SW44.1, SW45.1
- new net: SW46.1, SW47.1, SW48.1, SW49.1, SW50.1, SW51.1, SW52.1, SW53.1, SW54.1
- new net: SW55.1, SW56.1, SW57.1, SW58.1, SW59.1, SW60.1, SW61.1, SW62.1, SW63.1
- new net: SW64.1, SW65.1, SW66.1, SW67.1, SW68.1, SW69.1, SW70.1, SW71.1, SW72.1
- no-connect marks 5 -> 6
Other:
- moved on the sheet: J1, U1
