File: pcb/lasercut.kicad_pcb (KiCad board)
At the start: 2 copper layers, 338.6 x 105.3 mm, 159 parts, among them SW1 SW_Push, SW10 SW_Push, SW11 SW_Push, SW12 SW_Push, SW13 SW_Push, SW14 SW_Push, SW15 SW_Push, SW16 SW_Push, SW17 SW_Push, SW18 SW_Push, SW19 SW_Push, SW2 SW_Push, SW20 SW_Push, SW21 SW_Push, SW22 SW_Push, SW23 SW_Push, SW24 SW_Push, SW25 SW_Push, SW26 SW_Push, SW27 SW_Push, SW28 SW_Push, SW29 SW_Push, SW3 SW_Push, SW30 SW_Push, SW31 SW_Push, SW32 SW_Push, SW33 SW_Push, SW34 SW_Push, SW35 SW_Push, SW36 SW_Push, SW37 SW_Push, SW38 SW_Push, SW39 SW_Push, SW4 SW_Push, SW40 SW_Push, SW41 SW_Push, SW42 SW_Push, SW43 SW_Push, SW44 SW_Push, SW45 SW_Push, SW46 SW_Push, SW47 SW_Push, SW48 SW_Push, SW49 SW_Push, SW5 SW_Push, SW50 SW_Push, SW51 SW_Push, SW52 SW_Push, SW53 SW_Push, SW54 SW_Push, SW55 SW_Push, SW56 SW_Push, SW57 SW_Push, SW58 SW_Push, SW59 SW_Push, SW6 SW_Push, SW60 SW_Push, SW61 SW_Push, SW62 SW_Push, SW63 SW_Push, SW64 SW_Push, SW65 SW_Push, SW66 SW_Push, SW67 SW_Push, SW68 SW_Push, SW69 SW_Push, SW7 SW_Push, SW70 SW_Push, SW71 SW_Push, SW72 SW_Push, SW8 SW_Push, SW9 SW_Push

Commit message: FIX: Row5 was connected to GND
Parts:
- moved RESET 0.40 mm to (336.8, 88.0)
- renumbered REF** to BAT
Connections:
- U pad 2: (no net) -> ROW5
- U pad 3: (no net) -> GND
- U pad 4: ROW5 -> GND
Routing:
- net GND: track 16.2 -> 34.6 mm
- net ROW5: track 276.8 -> 284.1 mm
Changed lines of the file:
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@@
       (layerselection 0x00010fc_ffffffff)
       (disableapertmacros false)
-      (usegerberextensions false)
-      (usegerberattributes true)
-      (usegerberadvancedattributes true)
-      (creategerberjobfile true)
+      (usegerberextensions true)
+      (usegerberattributes false)
+      (usegerberadvancedattributes false)
+      (creategerberjobfile false)
       (svguseinch false)
       (svgprecision 6)
-      (excludeedgelayer true)
+      (excludeedgelayer false)
       (plotframeref false)
       (viasonmask false)
@@
       (plotinvisibletext false)
       (sketchpadsonfab false)
-      (subtractmaskfromsilk false)
+      (subtractmaskfromsilk true)
       (outputformat 1)
       (mirror false)
-      (drillshape 1)
+      (drillshape 0)
       (scaleselection 1)
-      (outputdirectory "")
+      (outputdirectory "gerber/")
     )
   )
@@
     (pad "1" thru_hole rect locked (at -13.97 7.62 180) (size 1.7526 1.7526) (drill 1.0922) (layers *.Cu *.SilkS *.Mask)
       (net 82 "ROW0"))
-    (pad "2" thru_hole circle locked (at -11.43 7.62 180) (size 1.7526 1.7526) (drill 1.0922) (layers *.Cu *.SilkS *.Mask))
-    (pad "3" thru_hole circle locked (at -8.89 7.62 180) (size 1.7526 1.7526) (drill 1.0922) (layers *.Cu *.SilkS *.Mask))
-    (pad "4" thru_hole circle locked (at -6.35 7.62 180) (size 1.7526 1.7526) (drill 1.0922) (layers *.Cu *.SilkS *.Mask)
+    (pad "2" thru_hole circle locked (at -11.43 7.62 180) (size 1.7526 1.7526) (drill 1.0922) (layers *.Cu *.SilkS *.Mask)
       (net 83 "ROW5"))
+    (pad "3" thru_hole circle locked (at -8.89 7.62 180) (size 1.7526 1.7526) (drill 1.0922) (layers *.Cu *.SilkS *.Mask)
+      (net 91 "GND"))
+    (pad "4" thru_hole circle locked (at -6.35 7.62 180) (size 1.7526 1.7526) (drill 1.0922) (layers *.Cu *.SilkS *.Mask)
+      (net 91 "GND"))
     (pad "5" thru_hole circle locked (at -3.81 7.62 180) (size 1.7526 1.7526) (drill 1.0922) (layers *.Cu *.SilkS *.Mask)
       (net 84 "ROW1"))
@@
   )
   (footprint "TestPoint:TestPoint_2Pads_Pitch2.54mm_Drill0.8mm" (layer "B.Cu")
-    (at 336.4 88 90)
+    (at 336.8 88 90)
     (descr "Test point with 2 pins, pitch 2.54mm, drill diameter 0.8mm")
     (tags "CONN DEV")
@@
     (tags "Through hole angled pin header THT 1x02 2.54mm single row")
     (attr through_hole)
-    (fp_text reference "REF**" (at 4.385 2.27 90) (layer "B.SilkS")
+    (fp_text reference "BAT" (at 4.385 2.27 90) (layer "B.SilkS")
       (effects (font (size 1 1) (thickness 0.15)) (justify mirror))
     )
@@
     (effects (font (size 1.5 1.5) (thickness 0.3)))
   )
-  (gr_text "RESET" (at 338.4 86.8 -270) (layer "F.SilkS")
+  (gr_text "RESET" (at 335.2 86.8 -270) (layer "F.SilkS")
     (effects (font (size 1 1) (thickness 0.15)))
   )
@@
   (segment (start 134.855 40.655) (end 153.905 40.655) (width 0.25) (layer "B.Cu") (net 82))
   (segment (start 351.50702 47.257027) (end 351.50702 62.84298) (width 0.25) (layer "B.Cu") (net 82))
-  (segment (start 344.145 40.655) (end 344.145 50.172013) (width 0.25) (layer "F.Cu") (net 83))
   (segment (start 344.145 50.172013) (end 341.75 52.567013) (width 0.25) (layer "F.Cu") (net 83))
-  (segment (start 341.75 52.567013) (end 341.75 64.98) (width 0.25) (layer "F.Cu") (net 83))
+  (segment (start 344.145 40.655) (end 344.145 50.172013) (width 0.25) (layer "F.Cu") (net 83))
+  (segment (start 341.75 52.567013) (end 341.75 59.9) (width 0.25) (layer "F.Cu") (net 83))
+  (segment (start 341.75 59.9) (end 346.83 64.98) (width 0.25) (layer "F.Cu") (net 83))
   (via (at 344.145 40.655) (size 0.8) (drill 0.4) (layers "F.Cu" "B.Cu") (net 83))
   (segment (start 344.145 40.655) (end 349.1675 40.655) (width 0.25) (layer "B.Cu") (net 83))
-  (segment (start 340.410811 66.319189) (end 341.75 64.98) (width 0.25) (layer "B.Cu") (net 83))
-  (segment (start 329.542989 117.429511) (end 350.570489 117.429511) (width 0.25) (layer "B.Cu") (net 83))
+  (segment (start 350.570489 117.429511) (end 351.6 116.4) (width 0.25) (layer "B.Cu") (net 83))
+  (segment (start 346.83 69.93) (end 346.83 64.98) (width 0.25) (layer "B.Cu") (net 83))
   (segment (start 328.913478 116.8) (end 329.542989 117.429511) (width 0.25) (layer "B.Cu") (net 83))
-  (segment (start 351.6 116.4) (end 351.6 103.8) (width 0.25) (layer "B.Cu") (net 83))
+  (segment (start 311.0675 116.855) (end 311.1225 116.8) (width 0.25) (layer "B.Cu") (net 83))
+  (segment (start 351.6 74.7) (end 346.83 69.93) (width 0.25) (layer "B.Cu") (net 83))
   (segment (start 211.055 40.655) (end 230.105 40.655) (width 0.25) (layer "B.Cu") (net 83))
-  (segment (start 350.570489 117.429511) (end 351.6 116.4) (width 0.25) (layer "B.Cu") (net 83))
-  (segment (start 351.6 103.8) (end 345.6 97.8) (width 0.25) (layer "B.Cu") (net 83))
-  (segment (start 345.6 97.8) (end 340.410811 92.610811) (width 0.25) (layer "B.Cu") (net 83))
   (segment (start 230.105 40.655) (end 249.155 40.655) (width 0.25) (layer "B.Cu") (net 83))
-  (segment (start 345.595 97.805) (end 330.1175 97.805) (width 0.25) (layer "B.Cu") (net 83))
+  (segment (start 329.542989 117.429511) (end 350.570489 117.429511) (width 0.25) (layer "B.Cu") (net 83))
   (segment (start 311.1225 116.8) (end 328.913478 116.8) (width 0.25) (layer "B.Cu") (net 83))
-  (segment (start 340.410811 92.610811) (end 340.410811 66.319189) (width 0.25) (layer "B.Cu") (net 83))
-  (segment (start 311.0675 116.855) (end 311.1225 116.8) (width 0.25) (layer "B.Cu") (net 83))
+  (segment (start 345.595 97.805) (end 330.1175 97.805) (width 0.25) (layer "B.Cu") (net 83))
+  (segment (start 351.6 116.4) (end 351.6 74.7) (width 0.25) (layer "B.Cu") (net 83))
   (segment (start 249.155 40.655) (end 268.205 40.655) (width 0.25) (layer "B.Cu") (net 83))
   (segment (start 296.78 40.655) (end 330.1175 40.655) (width 0.25) (layer "B.Cu") (net 83))
   (segment (start 330.1175 40.655) (end 344.145 40.655) (width 0.25) (layer "B.Cu") (net 83))
   (segment (start 268.205 40.655) (end 296.78 40.655) (width 0.25) (layer "B.Cu") (net 83))
-  (segment (start 345.6 97.8) (end 345.595 97.805) (width 0.25) (layer "B.Cu") (net 83))
+  (segment (start 351.6 91.8) (end 345.595 97.805) (width 0.25) (layer "B.Cu") (net 83))
   (segment (start 163.43 59.705) (end 182.48 59.705) (width 0.25) (layer "B.Cu") (net 84))
   (segment (start 289.120489 60.279511) (end 293.504511 55.895489) (width 0.25) (layer "B.Cu") (net 84))
@@
   (segment (start 344.99 84.6) (end 349.37 80.22) (width 0.35) (layer "B.Cu") (net 90))
   (segment (start 346.83 84.57) (end 346.8 84.6) (width 0.35) (layer "F.Cu") (net 91))
-  (segment (start 343.4 88) (end 336.4 88) (width 0.35) (layer "F.Cu") (net 91))
+  (segment (start 343.4 88) (end 336.8 88) (width 0.35) (layer "F.Cu") (net 91))
   (segment (start 346.83 80.22) (end 346.83 84.57) (width 0.35) (layer "F.Cu") (net 91))
   (segment (start 346.8 84.6) (end 343.4 88) (width 0.35) (layer "F.Cu") (net 91))
+  (segment (start 344.29 64.98) (end 344.29 77.68) (width 0.35) (layer "B.Cu") (net 91))
+  (segment (start 341.75 64.98) (end 344.29 64.98) (width 0.35) (layer "B.Cu") (net 91))
+  (segment (start 344.29 77.68) (end 346.83 80.22) (width 0.35) (layer "B.Cu") (net 91))
   (segment (start 344.29 80.22) (end 339.05 85.46) (width 0.25) (layer "F.Cu") (net 92))
-  (segment (start 339.05 85.46) (end 336.4 85.46) (width 0.25) (layer "F.Cu") (net 92))
+  (segment (start 339.05 85.46) (end 336.8 85.46) (width 0.25) (layer "F.Cu") (net 92))
   (group "" locked (id a91b8a04-3400-4136-bdcc-9e2b2d30d4e0)
     (members

Commit message: 90% re routed
Parts:
- removed REF**: OSHW-Logo_5.7x6mm_Copper, Symbol:OSHW-Logo_5.7x6mm_Copper
- moved U 2.24 mm to (333.4, 71.6)
Connections:
- D30 pad 1: ROW7 -> ROW6
- D59 pad 1: ROW6 -> ROW7
- U pad 1: ROW0 -> (no net)
- U pad 10: ROW4 -> COL1
- U pad 12: COL1 -> ROW1
- U pad 13: COL2 -> COL8
- U pad 14: COL3 -> ROW7
- U pad 15: COL4 -> ROW4
- U pad 16: COL5 -> ROW3
- U pad 17: COL6 -> ROW2
- U pad 18: COL7 -> ROW0
- U pad 19: COL8 -> COL6
- U pad 2: ROW5 -> COL7
- U pad 20: (no net) -> COL5
- U pad 21: (no net) -> VCC
- U pad 5: ROW1 -> (no net)
- U pad 7: ROW7 -> COL4
- U pad 8: ROW2 -> COL3
- U pad 9: ROW3 -> COL2
Routing:
- net COL4: track 566.5 -> 393.3 mm
- net ROW5: track 284.1 -> 169.6 mm, vias 1 -> 0
- net ROW6: track 256.1 -> 162.5 mm, vias 1 -> 0
- net COL6: track 433.5 -> 340.4 mm
- net GND: track 34.6 -> 0.00 mm
- net COL7: track 317.5 -> 285.7 mm
- net COL5: track 432.9 -> 406.3 mm, vias 0 -> 2
- net ROW7: track 198.8 -> 221.7 mm, vias 0 -> 4
- net ROW3: track 322.8 -> 300.8 mm, vias 1 -> 0
- net ROW1: track 300.7 -> 283.0 mm
- net ROW0: track 335.5 -> 320.2 mm
- net ROW2: track 290.5 -> 302.0 mm
- net COL0: track 413.1 -> 423.0 mm, vias 0 -> 1
- net RST: track 9.66 -> 0.00 mm
- net COL8: track 268.3 -> 260.5 mm, vias 0 -> 1
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Other:
- board text removed: "Lasercut v1.0 lad1337 03/2022"
- board text removed: "RESET"
